Commit message: retrain sdog with perfect gait? remember to fix the joint limit in the xml file sim to sim still fail maybe xml has problem and some test to test mujoco and isaac

File: resources/robots/sdog/urdf/sdog.urdf (robot description, URDF)
Before this commit: robot sdog, 18 links, 17 joints
Joints:
- joint bl_hip_joint: limit lower=-0.8 upper=0.8 effort=0.45 velocity=10 -> lower=-0.3 upper=0.3 effort=0.45 velocity=10
- joint br_hip_joint: limit lower=-0.8 upper=0.8 effort=0.45 velocity=10 -> lower=-0.3 upper=0.3 effort=0.45 velocity=10
- joint fl_hip_joint: limit lower=-0.8 upper=0.8 effort=0.45 velocity=10 -> lower=-0.3 upper=0.3 effort=0.45 velocity=10
- joint fr_hip_joint: limit lower=-0.8 upper=0.8 effort=0.45 velocity=10 -> lower=-0.3 upper=0.3 effort=0.45 velocity=10
